File: projects/oph/pcb/OPH Driver Mk 2.kicad_pcb (KiCad board)
At the start: 4 copper layers, 147.9 x 80 mm, 210 parts, among them M1 MT-HOLE, M2 MT-HOLE, M3 MT-HOLE, M4 MT-HOLE, P1 USB-MICRO-B, P10 5V, P11 4.096V, P12 1V7, P13 A5V, P14 3V3, P15 -12V, P16 CM+, P17 AGND, P18 MD, P19 ADC_SDI, P2 SP0, P20 ADC_SCK, P21 ADC_SDO, P22 ADC_CNV, P23 ADC+, P24 CM-, P25 ADC-, P26 I+, P27 I-, P28 FES, P29 c, P3 SP1, P30 d, P31 a, P32 b, P33 MOLEX 054550-2671, P34 c-d, P35 F_SCLK, P36 F_DIN, P37 F_SYNC, P38 FO-, P39 FO+, P4 SP2, P40 FOCUS, P41 T_SCLK, P42 T_DIN, P43 T_SYNC, P44 TRACK, P45 TO+, P46 TO-, P47 GND, P48 GND, P49 GND, P5 SP3, P50 GND, P51 DACREF, P52 -5V, P6 SP4, P7 VIN, P8 2.5mm DC JACK, P9 +12V, Q1 MMBT3904, U1 FT232R, U10 AD7691, U11 IC-WKM, U12 ADA4941-1, U13 AD8222, U14 AD5062, U15 TLV4120, U16 AD5062, U17 TLV4120, U18 ADR4540, U19 LT1677, U2 24LC256, U20 LT1677, U21 LT1677, U3 P8X32A, U4 TEN5-1222, U5 TEN5-1211, U6 ADR4540, U7 TPS7A4901, U8 SPX3819, U9 TPS7A3001, X1 8MHz

Commit message: oph v2 updates
Parts:
- R17: value 1k -> 330R
- moved R17 3.19 mm to (180.2, 189.4), turned to 180 degrees
- moved C37 1.63 mm to (239.4, 166.8), turned to 270 degrees
- moved C38 0.84 mm to (240.9, 166.8), turned to 270 degrees
Connections:
- C10 pad 1: N-0000091 -> Net-(C10-Pad1)
- C11 pad 1: N-0000091 -> Net-(C10-Pad1)
- C12 pad 1: N-0000091 -> Net-(C10-Pad1)
- C9 pad 1: N-0000091 -> Net-(C10-Pad1)
- D6 pad 2: GNDPWR -> GND
- M1 pad 0: (no net) -> Net-(M1-Pad0)
- M2 pad 0: (no net) -> Net-(M2-Pad0)
- M3 pad 0: (no net) -> Net-(M3-Pad0)
- M4 pad 0: (no net) -> Net-(M4-Pad0)
- P1 pad 0: (no net) -> Net-(P1-Pad0)
- P1 pad 4: (no net) -> Net-(P1-Pad4)
- P33 pad 12: (no net) -> Net-(P33-Pad12)
- P33 pad 13: (no net) -> Net-(P33-Pad13)
- P33 pad 16: (no net) -> Net-(P33-Pad16)
- P33 pad 17: (no net) -> Net-(P33-Pad17)
- P33 pad 19: (no net) -> Net-(P33-Pad19)
- P33 pad 20: (no net) -> Net-(P33-Pad20)
- P33 pad 21: (no net) -> Net-(P33-Pad21)
- P33 pad 23: (no net) -> Net-(P33-Pad23)
- P33 pad 24: (no net) -> Net-(P33-Pad24)
- P33 pad 7: (no net) -> Net-(P33-Pad7)
- P33 pad 8: (no net) -> Net-(P33-Pad8)
- P7 pad 1: N-0000091 -> Net-(C10-Pad1)
- P8 pad 3: N-0000091 -> Net-(C10-Pad1)
- R17 pad 2: N-0000091 -> 3V3
- RV2 pad 3: (no net) -> 4VR
- U1 pad 10: (no net) -> Net-(U1-Pad10)
- U1 pad 11: (no net) -> Net-(U1-Pad11)
- U1 pad 12: (no net) -> Net-(U1-Pad12)
- U1 pad 13: (no net) -> Net-(U1-Pad13)
- U1 pad 14: (no net) -> Net-(U1-Pad14)
- U1 pad 19: (no net) -> Net-(U1-Pad19)
- U1 pad 27: (no net) -> Net-(U1-Pad27)
- U1 pad 28: (no net) -> Net-(U1-Pad28)
- U1 pad 3: (no net) -> Net-(U1-Pad3)
- U1 pad 6: (no net) -> Net-(U1-Pad6)
- U1 pad 9: (no net) -> Net-(U1-Pad9)
- U11 pad 4: (no net) -> Net-(U11-Pad4)
- U12 pad 7: (no net) -> Net-(U12-Pad7)
- U13 pad 10: (no net) -> Net-(U13-Pad10)
- U13 pad 11: (no net) -> Net-(U13-Pad11)
- U13 pad 2: (no net) -> Net-(U13-Pad2)
- U13 pad 3: (no net) -> Net-(U13-Pad3)
- U19 pad 1: (no net) -> Net-(U19-Pad1)
- U19 pad 8: (no net) -> Net-(U19-Pad8)
- U20 pad 1: (no net) -> Net-(U20-Pad1)
- U20 pad 8: (no net) -> Net-(U20-Pad8)
- U21 pad 1: (no net) -> Net-(U21-Pad1)
- U21 pad 8: (no net) -> Net-(U21-Pad8)
- U3 pad 10: (no net) -> Net-(U3-Pad10)
- U3 pad 11: (no net) -> Net-(U3-Pad11)
- U3 pad 12: (no net) -> Net-(U3-Pad12)
- U3 pad 2: (no net) -> Net-(U3-Pad2)
- U3 pad 21: (no net) -> Net-(U3-Pad21)
- U3 pad 22: (no net) -> Net-(U3-Pad22)
- U3 pad 23: (no net) -> Net-(U3-Pad23)
- U3 pad 24: (no net) -> Net-(U3-Pad24)
- U3 pad 25: (no net) -> Net-(U3-Pad25)
- U3 pad 26: (no net) -> Net-(U3-Pad26)
- U3 pad 3: (no net) -> Net-(U3-Pad3)
- U3 pad 9: (no net) -> Net-(U3-Pad9)
- U4 pad 22: N-0000091 -> Net-(C10-Pad1)
- U4 pad 23: N-0000091 -> Net-(C10-Pad1)
- U5 pad 22: N-0000091 -> Net-(C10-Pad1)
- U5 pad 23: N-0000091 -> Net-(C10-Pad1)
Routing:
- net 1V7: track 15.1 -> 35.0 mm
- net Net-(P30-Pad1): track 18.4 -> 2.98 mm, vias 1 -> 0
- net Net-(D6-Pad1): track 0.00 -> 3.87 mm
- net 4VR: track 0.00 -> 1.94 mm, vias 0 -> 2
- net (no net): track 1.94 -> 0.00 mm, vias 2 -> 0
- net ADC_SDI: track 69.9 -> 71.0 mm
- net GND: track 173.5 -> 174.5 mm, vias 155 -> 156
- net GNDPWR: track 126.0 -> 125.1 mm, vias 47 -> 46
- net 3V3: track 33.3 -> 32.4 mm
- added copper zone on GND, net GND
- added copper zone on GND, net GNDPWR
- added copper zone on F.Cu, net N-0000092
- added copper zone on F.Cu, net N-0000094
- removed copper zone on F.Cu, net +5V
- removed copper zone on F.Cu, net -5V
- removed copper zone on B.Cu, net GNDPWR
- removed copper zone on F.Cu, net Net-(C13-Pad1)
- removed copper zone on F.Cu, net Net-(C14-Pad2)
