File: projects/oph/pcb/Power and references.sch (KiCad schematic (older format))
At the start: 56 parts, among them P10 5V, P11 4.096V, P12 1V7, P13 A5V, P14 3V3, P15 -12V, P51 DACREF, P52 -5V, P7 VIN, P8 2.5mm DC JACK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

Commit message: oph v2 updates
Parts:
- R17: value 1k -> 330R
Connections:
- net 3V3: now also R17.2
- net GND: now also D6.2 (K)
- net GNDPWR: no longer D6.2 (K)
- net at C10.1, C11.1, C12.1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: no longer R17.2
Other:
- moved on the sheet: D6, R17
Changed lines of the file:
@@
 LIBS:valves
 LIBS:OPH Driver Mk 2-cache
-EELAYER 27 0
+EELAYER 24 0
 EELAYER END
 $Descr A3 16535 11693
@@
 	1    0    0    -1
 $EndComp
-Text Notes 3825 4900 0    80   ~ 0
+Text Notes 3700 5000 0    80   ~ 0
 5V SUPPLY FOR MCU \nAND FOCUS/TRACKING
 Text Notes 9475 2425 0    80   ~ 0
@@
 L LED D6
 U 1 1 51D93077
-P 2350 3650
-F 0 "D6" V 2275 3500 50  0000 C CNN
-F 1 "'ON'" V 2350 3500 50  0000 C CNN
-F 2 "~" H 2350 3650 60  0000 C CNN
-F 3 "~" H 2350 3650 60  0000 C CNN
-	1    2350 3650
-	0    1    1    0
+P 8950 6100
+F 0 "D6" V 8875 5950 50  0000 C CNN
+F 1 "'ON'" V 8950 5950 50  0000 C CNN
+F 2 "~" H 8950 6100 60  0000 C CNN
+F 3 "~" H 8950 6100 60  0000 C CNN
+	1    8950 6100
+	0    -1   1    0
 $EndComp
 $Comp
 L R R17
 U 1 1 51D93088
-P 2650 3400
-F 0 "R17" V 2825 3400 50  0000 C CNN
-F 1 "1k" V 2750 3400 50  0000 C CNN
-F 2 "~" V 2580 3400 30  0000 C CNN
-F 3 "~" H 2650 3400 30  0000 C CNN
-	1    2650 3400
-	0    -1   -1   0
+P 8650 5850
+F 0 "R17" V 8825 5850 50  0000 C CNN
+F 1 "330R" V 8750 5850 50  0000 C CNN
+F 2 "~" V 8580 5850 30  0000 C CNN
+F 3 "~" H 8650 5850 30  0000 C CNN
+	1    8650 5850
+	0    1    -1   0
 $EndComp
 $Comp
@@
 	5950 5850 6800 5850
 Wire Wire Line
-	2350 3850 2350 3925
+	8950 6300 8950 6375
 Wire Wire Line
 	2850 2850 2850 3050
@@
 Connection ~ 8425 3250
 Wire Wire Line
-	7700 5850 8300 5850
-Wire Wire Line
-	2400 3400 2350 3400
-Wire Wire Line
-	2350 3400 2350 3450
-Wire Wire Line
-	2900 3400 3000 3400
-Connection ~ 3000 3400
+	7700 5850 8400 5850
+Wire Wire Line
+	8900 5850 8950 5850
+Wire Wire Line
+	8950 5850 8950 5900
 $Comp
 L TST P9
@@
 $Comp
 L GNDPWR #PWR?
-U 1 1 53D4798D
-P 2350 3925
-F 0 "#PWR?" H 2350 3975 40  0001 C CNN
-F 1 "GNDPWR" H 2350 3845 40  0000 C CNN
-F 2 "" H 2350 3925 60  0000 C CNN
-F 3 "" H 2350 3925 60  0000 C CNN
-	1    2350 3925
-	1    0    0    -1
-$EndComp
-$Comp
-L GNDPWR #PWR?
 U 1 1 53D47993
 P 3500 4450
@@
 	1    0    0    -1
 $EndComp
+$Comp
+L GND #PWR?
+U 1 1 5419506F
+P 8950 6375
+F 0 "#PWR?" H 8950 6375 30  0001 C CNN
+F 1 "GND" H 8950 6305 30  0001 C CNN
+F 2 "" H 8950 6375 60  0000 C CNN
+F 3 "" H 8950 6375 60  0000 C CNN
+	1    8950 6375
+	1    0    0    -1
+$EndComp
+Connection ~ 8300 5850
 $EndSCHEMATC
